Commit message: Modified reward.

File: src/omni_3wd/urdf/main.urdf.xacro (robot description, xacro)
@@ -125,5 +125,5 @@
     		<parent link="plate_1_link"/>
     		<child link="base_scan"/>
-    		<origin xyz="-0.0 0 0.028" rpy="0 0 0"/>
+    		<origin xyz="-0.0 0 0.028" rpy="0 0 -0.52"/>
   	</joint>
 	<link name="base_scan">

Commit message: update

File: src/omni_3wd/urdf/main.urdf.xacro (robot description, xacro)
@@ -125,5 +125,5 @@
     		<parent link="plate_1_link"/>
     		<child link="base_scan"/>
-    		<origin xyz="-0.0 0 0.028" rpy="0 0 -0.52"/>
+    		<origin xyz="-0.0 0 0.028" rpy="0 0 0"/>
   	</joint>
 	<link name="base_scan">

Commit message: Workaround :Odom topic stops working after reset gazebo enviroment.

File: src/omni_3wd/urdf/main.urdf.xacro (robot description, xacro)
@@ -19,5 +19,15 @@
     	<xacro:property name="standoff_y" value="0.10"/>
 	<!-- Define Base -->
-	<link name="origin_link"/>
+	<!--link name="base_footprint"-->
+	<!--link name="origin_link"/-->
+	<!-- root link, on the ground just below the model origin -->
+	<link name="base_footprint">
+	<visual>
+		<origin xyz="0 0 0" rpy="0 0 0" />
+		<geometry>
+			<box size="0.001 0.001 0.001" />
+		</geometry>
+		</visual>
+	</link>
 	<link name="base_link">
 	<inertial>
@@ -46,5 +56,5 @@
 	</link>
 	<joint name="base_joint" type="fixed">
-		<parent link="origin_link" />
+		<parent link="base_footprint" />
 		<child link="base_link" />
 		<origin xyz="0 0 0.01905"/>
@@ -170,5 +180,5 @@
   	</gazebo>
 	<gazebo reference="rim_left_link">
-    		<material>Gazebo/Gray</material>
+    		<material>Gazebo/Blue</material>
   	</gazebo>
 	<gazebo reference="rim_back_link">
@@ -176,5 +186,5 @@
   	</gazebo>
 	<gazebo reference="rim_right_link">
-    		<material>Gazebo/Gray</material>
+    		<material>Gazebo/Green</material>
   	</gazebo>
 	<gazebo reference="standoff_2in_1_link">
@@ -194,18 +204,59 @@
   	</gazebo>
 	<!-- Add controller system plugin -->
-	<!--gazebo>
+	<!--
+	<gazebo>
 		<plugin name="gazebo_ros_control" filename="libgazebo_ros_control.so">
 		<robotNamespace>/open_base</robotNamespace>
 		</plugin>
-	</gazebo-->
+	</gazebo>
+	-->
 	<!-- Add controller system plugin -->
 	<gazebo>
 		<plugin name="object_controller" filename="libgazebo_ros_planar_move.so">
 		<commandTopic>cmd_vel</commandTopic>
+		<!--odometryTopic>odom</odometryTopic-->
+		<!--odometryFrame>odom</odometryFrame-->
+		<!--odometryRate>20.0</odometryRate-->
+		<robotBaseFrame>base_footprint</robotBaseFrame>
+		</plugin>
+	</gazebo>
+	<!-- Workaround :
+		Use the object_controller only can not get the odom data which will stop working ,
+		So I add the differential_drive_controller for getting the odom data. -->
+	<gazebo>
+	<plugin name="differential_drive_controller" filename="libgazebo_ros_diff_drive.so">
+		<!-- Plugin update rate in Hz -->
+		<updateRate>20</updateRate>
+		<!-- Name of left joint, defaults to `left_joint` -->
+		<leftJoint>rim_right_joint</leftJoint>
+		<!-- Name of right joint, defaults to `right_joint` -->
+		<rightJoint>rim_back_joint</rightJoint>
+		<!-- The distance from the center of one wheel to the other, in meters, defaults to 0.34 m -->
+		<!--wheelSeparation>0.2078461</wheelSeparation-->
+		<!-- Diameter of the wheels, in meters, defaults to 0.15 m -->
+		<!--wheelDiameter>0.114</wheelDiameter-->
+		<!-- Wheel acceleration, in rad/s^2, defaults to 0.0 rad/s^2 -->
+		<!--wheelAcceleration>1.0</wheelAcceleration-->
+		<!-- Maximum torque which the wheels can produce, in Nm, defaults to 5 Nm -->
+		<!--wheelTorque>20</wheelTorque-->
+		<!-- Topic to receive geometry_msgs/Twist message commands, defaults to `cmd_vel` -->
+		<!--commandTopic>cmd_vel</commandTopic-->
+		<!-- Topic to publish nav_msgs/Odometry messages, defaults to `odom` -->
 		<odometryTopic>odom</odometryTopic>
+		<!-- Odometry frame, defaults to `odom` -->
 		<odometryFrame>odom</odometryFrame>
-		<odometryRate>20.0</odometryRate>
-		<robotBaseFrame>base_link</robotBaseFrame>
-		</plugin>
+		<!-- Robot frame to calculate odometry from, defaults to `base_footprint` -->
+		<robotBaseFrame>base_footprint</robotBaseFrame>
+		<!-- Odometry source, 0 for ENCODER, 1 for WORLD, defaults to WORLD -->
+		<odometrySource>1</odometrySource>
+		<!-- Set to true to publish transforms for the wheel links, defaults to false -->
+		<publishWheelTF>true</publishWheelTF>
+		<!-- Set to true to publish transforms for the odometry, defaults to true -->
+		<publishOdom>true</publishOdom>
+		<!-- Set to true to publish sensor_msgs/JointState on /joint_states for the wheel joints, defaults to false -->
+		<publishWheelJointState>true</publishWheelJointState>
+		<!-- Set to true to swap right and left wheels, defaults to true -->
+		<legacyMode>false</legacyMode>
+	</plugin>
 	</gazebo>
 	<!-- Add plugin for calculate position and Vx Vy Vz -->
@@ -223,4 +274,5 @@
 	</gazebo-->
 	<!-- Add IMU Controller Plugin -->
+	<!--
 	<gazebo reference="imu_link">
 	    <sensor type="imu" name="imu">
@@ -230,4 +282,5 @@
 	    <material>Gazebo/FlatBlack</material>
 	</gazebo>
+	-->
 	<!-- Add IMU Controller Plugin , no gravity -->
 	<!--gazebo>
@@ -264,5 +317,5 @@
 		<sensor name="imu_sensor" type="imu">
 		<always_on>true</always_on>
-		<update_rate>100</update_rate>
+		<!--update_rate>100</update_rate-->
 		<visualize>true</visualize>
 		<topic>__default_topic__</topic>
@@ -270,5 +323,9 @@
 			<topicName>imu</topicName>
 			<bodyName>imu_link</bodyName>
-			<updateRateHZ>10.0</updateRateHZ>
+			<!--updateRateHZ>10.0</updateRateHZ-->
+			<!--set the update rate will broken the imu topic after reset gazebo env
+			,set it to zero will make it normal.
+			https://github.com/ros-simulation/gazebo_ros_pkgs/issues/169-->
+			<updateRateHZ>0.0</updateRateHZ>
 			<gaussianNoise>0.0</gaussianNoise>
 			<xyzOffset>0 0 0</xyzOffset>

Commit message: Try to integrate slam pakage.

File: src/omni_3wd/urdf/main.urdf.xacro (robot description, xacro)
@@ -19,7 +19,7 @@
     	<xacro:property name="standoff_y" value="0.10"/>
 	<!-- Define Base -->
-	<!--link name="base_footprint"-->
-	<!--link name="origin_link"/-->
+	<link name="base_footprint"/>
 	<!-- root link, on the ground just below the model origin -->
+	<!--
 	<link name="base_footprint">
 	<visual>
@@ -30,4 +30,5 @@
 		</visual>
 	</link>
+	-->
 	<link name="base_link">
 	<inertial>
@@ -215,7 +216,7 @@
 		<plugin name="object_controller" filename="libgazebo_ros_planar_move.so">
 		<commandTopic>cmd_vel</commandTopic>
-		<!--odometryTopic>odom</odometryTopic-->
-		<!--odometryFrame>odom</odometryFrame-->
-		<!--odometryRate>20.0</odometryRate-->
+		<odometryTopic>odom</odometryTopic>
+		<odometryFrame>odom</odometryFrame>
+		<odometryRate>20.0</odometryRate>
 		<robotBaseFrame>base_footprint</robotBaseFrame>
 		</plugin>
@@ -232,14 +233,14 @@
 		<!-- Name of right joint, defaults to `right_joint` -->
 		<rightJoint>rim_back_joint</rightJoint>
-		<!-- The distance from the center of one wheel to the other, in meters, defaults to 0.34 m -->
-		<!--wheelSeparation>0.2078461</wheelSeparation-->
-		<!-- Diameter of the wheels, in meters, defaults to 0.15 m -->
-		<!--wheelDiameter>0.114</wheelDiameter-->
-		<!-- Wheel acceleration, in rad/s^2, defaults to 0.0 rad/s^2 -->
-		<!--wheelAcceleration>1.0</wheelAcceleration-->
-		<!-- Maximum torque which the wheels can produce, in Nm, defaults to 5 Nm -->
-		<!--wheelTorque>20</wheelTorque-->
-		<!-- Topic to receive geometry_msgs/Twist message commands, defaults to `cmd_vel` -->
-		<!--commandTopic>cmd_vel</commandTopic-->
+			<!-- The distance from the center of one wheel to the other, in meters, defaults to 0.34 m -->
+			<!--wheelSeparation>0.2078461</wheelSeparation-->
+			<!-- Diameter of the wheels, in meters, defaults to 0.15 m -->
+			<!--wheelDiameter>0.114</wheelDiameter-->
+			<!-- Wheel acceleration, in rad/s^2, defaults to 0.0 rad/s^2 -->
+			<!--wheelAcceleration>1.0</wheelAcceleration-->
+			<!-- Maximum torque which the wheels can produce, in Nm, defaults to 5 Nm -->
+			<!--wheelTorque>20</wheelTorque-->
+			<!-- Topic to receive geometry_msgs/Twist message commands, defaults to `cmd_vel` -->
+			<!--commandTopic>cmd_vel</commandTopic-->
 		<!-- Topic to publish nav_msgs/Odometry messages, defaults to `odom` -->
 		<odometryTopic>odom</odometryTopic>
@@ -250,8 +251,9 @@
 		<!-- Odometry source, 0 for ENCODER, 1 for WORLD, defaults to WORLD -->
 		<odometrySource>1</odometrySource>
-		<!-- Set to true to publish transforms for the wheel links, defaults to false -->
-		<publishWheelTF>true</publishWheelTF>
+			<!-- Set to true to publish transforms for the wheel links, defaults to false -->
+			<!--publishWheelTF>true</publishWheelTF-->
 		<!-- Set to true to publish transforms for the odometry, defaults to true -->
-		<publishOdom>true</publishOdom>
+		<publishOdom>false</publishOdom>
+		<publishOdomTF>true</publishOdomTF>
 		<!-- Set to true to publish sensor_msgs/JointState on /joint_states for the wheel joints, defaults to false -->
 		<publishWheelJointState>true</publishWheelJointState>
@@ -343,5 +345,5 @@
 	      <pose>0 0 0 0 0 0</pose>
 	      <visualize>$(arg laser_visual)</visualize>
-	      <update_rate>5</update_rate>
+	      <update_rate>10</update_rate>
 	      <ray>
 		<scan>

Commit message: Fix some bugs.And rename the launch file.

File: src/omni_3wd/urdf/main.urdf.xacro (robot description, xacro)
@@ -32,27 +32,28 @@
 	-->
 	<link name="base_link">
-	<inertial>
-		<mass value="2.12299505415"/>
-		<inertia
-			ixx="0.00494744483"
-			ixy="0"
-			ixz="0"
-			iyy="0.00494744483"
-			iyz="0"
-			izz="0.00958868684"/>
-		</inertial>
-	<visual>
-		<geometry>
-			<mesh filename="package://omni_3wd/mesh/base.stl" scale="3.0 3.0 3.0"/>
-		</geometry>
-		<material name="base_material">
-			<color rgba="1 1 1 1"/>
-		</material>
-	</visual>
-	<collision>
-		<geometry>
-			<mesh filename="package://omni_3wd/mesh/base.stl" scale="3.0 3.0 3.0"/>
-		</geometry>
-	</collision>
+		<gravity>true</gravity>
+		<inertial>
+			<mass value="2.12299505415"/>
+			<inertia
+				ixx="0.00494744483"
+				ixy="0"
+				ixz="0"
+				iyy="0.00494744483"
+				iyz="0"
+				izz="0.00958868684"/>
+			</inertial>
+		<visual>
+			<geometry>
+				<mesh filename="package://omni_3wd/mesh/base.stl" scale="3.0 3.0 3.0"/>
+			</geometry>
+			<material name="base_material">
+				<color rgba="1 1 1 1"/>
+			</material>
+		</visual>
+		<collision>
+			<geometry>
+				<mesh filename="package://omni_3wd/mesh/base.stl" scale="3.0 3.0 3.0"/>
+			</geometry>
+		</collision>
 	</link>
 	<joint name="base_joint" type="fixed">
@@ -104,9 +105,10 @@
         </joint>
         <link name="plate_1_link">
+			<gravity>true</gravity>
             <inertial>
-                <mass value="0.1" />
+                <mass value="1.0" />
                 <origin xyz="0 0 0" />
-                <inertia ixx="0.01" ixy="0.0" ixz="0.0"
-                         iyy="0.01" iyz="0.0" izz="0.01" />
+                <inertia ixx="0.16" ixy="0.0" ixz="0.0"
+                         iyy="0.16" iyz="0.0" izz="0.16" />
             </inertial>
             <visual>
@@ -349,5 +351,5 @@
 		<scan>
 		  <horizontal>
-		    <samples>24</samples>
+		    <samples>360</samples>
 		    <resolution>1</resolution>
 		    <min_angle>0.0</min_angle>

File: src/omni_3wd/urdf/rim.urdf.xacro (robot description, xacro)
@@ -6,4 +6,5 @@
 	params="name color xyz rpy">
 		<link name="rim_${name}_link">
+			<gravity>true</gravity>
 			<inertial>
 				<origin xyz="0 0 -0.001029"/>
